File: boards/SIC431/SIC431/SIC431.kicad_sch (KiCad schematic)
At the start: 83 parts, among them J101 Screw_Terminal_01x02, J102 Screw_Terminal_01x06, J103 Screw_Terminal_01x06, J104 Screw_Terminal_01x06, K101 Relay, K102 Relay, K103 Relay, K104 Relay, K105 Relay, K106 Relay, SW101 SW_Push_Open, U101 SIC431AED-T1-GE3, U102 SIC431AED-T1-GE3, U103 SIC431AED-T1-GE3

Commit message: update on E-stop
Parts:
- SW101: footprint (none) -> power_board_support:E-Stop
Connections:
- net V_BAT_IN: now also K101.1, K102.1, K103.1, K104.1, K105.1, K106.1
- net 12V renamed E-stop
- net E-stop: no longer K101.1, K102.1, K103.1, K104.1, K105.1, K106.1

Commit message: update
Connections:
- net Earth is gone; now on net GND: C101.2, C102.2, C103.2, C104.2, C105.2, C106.2, C110.2, C111.2, C112.2, C116.2, C117.2, C118.2, C119.2, C120.2, C121.2, R102.2, R104.2, R106.2, U101.13 (PGND), U101.27_1 (PGND), U101.27_2 (PGND), U101.3 (PGND), U101.4 (PGND), U102.13 (PGND), U102.27_1 (PGND), U102.27_2 (PGND), U102.3 (PGND), U102.4 (PGND), U103.13 (PGND), U103.27_1 (PGND), U103.27_2 (PGND), U103.3 (PGND), U103.4 (PGND)
- net at C116.1, C119.1, L101.2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: now also D108.1 (A)
- net at C117.1, C120.1, L102.2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: now also D107.1 (A)

Commit message: updates
Parts:
- added J105, J106, J107: Conn_02x02_Top_Bottom, power_board_support:LM2596, symbol Connector_Generic:Conn_02x02_Top_Bottom
- added J108, J109, J110: Screw_Terminal_01x02, Connector_PinHeader_2.54mm:PinHeader_1x02_P2.54mm_Vertical, symbol Connector:Screw_Terminal_01x02
- C101, C102, C103: footprint Capacitor_SMD:C_0805_2012Metric -> Capacitor_THT:CP_Radial_D12.5mm_P5.00mm
Connections:
- net 5V_OUT_1: now also J108.1 (Pin_1)
- net 5V_OUT_2: now also J107.3 (Pin_3), J109.1 (Pin_1)
- net 5V_OUT_3: now also J106.3 (Pin_3), J110.1 (Pin_1)
- net GND: now also J105.2 (Pin_2), J105.4 (Pin_4), J106.2 (Pin_2), J106.4 (Pin_4), J107.2 (Pin_2), J107.4 (Pin_4), J108.2 (Pin_2), J109.2 (Pin_2), J110.2 (Pin_2)
- net V_BAT_IN: now also J105.1 (Pin_1), J106.1 (Pin_1), J107.1 (Pin_1)
Other:
- note added: "Backup 5 Volt Regulators"

Commit message: mostly complete
Parts:
- J105, J106, J107: footprint power_board_support:LM2596 -> power_board_support:LM2596-2
Changed lines of the file:
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@@
     (property "Reference" "J105" (id 0) (at 286.004 164.5625 0))
     (property "Value" "Conn_02x02_Top_Bottom" (id 1) (at 286.004 167.3376 0))
-    (property "Footprint" "power_board_support:LM2596" (id 2) (at 284.734 169.799 0)
+    (property "Footprint" "power_board_support:LM2596-2" (id 2) (at 284.734 169.799 0)
       (effects (font (size 1.27 1.27)) hide)
     )
@@
     (property "Reference" "J106" (id 0) (at 286.004 207.3615 0))
     (property "Value" "Conn_02x02_Top_Bottom" (id 1) (at 286.004 210.1366 0))
-    (property "Footprint" "power_board_support:LM2596" (id 2) (at 284.734 212.598 0)
+    (property "Footprint" "power_board_support:LM2596-2" (id 2) (at 284.734 212.598 0)
       (effects (font (size 1.27 1.27)) hide)
     )
@@
     (property "Reference" "J107" (id 0) (at 286.131 182.9775 0))
     (property "Value" "Conn_02x02_Top_Bottom" (id 1) (at 286.131 185.7526 0))
-    (property "Footprint" "power_board_support:LM2596" (id 2) (at 284.861 188.214 0)
+    (property "Footprint" "power_board_support:LM2596-2" (id 2) (at 284.861 188.214 0)
       (effects (font (size 1.27 1.27)) hide)
     )
@@
     )
     (path "/be8a1446-c460-4ce8-8c5a-a6e97ca6fc24"
-      (reference "J105") (unit 1) (value "Conn_02x02_Top_Bottom") (footprint "power_board_support:LM2596")
+      (reference "J105") (unit 1) (value "Conn_02x02_Top_Bottom") (footprint "power_board_support:LM2596-2")
     )
     (path "/c846d084-ce0f-49f0-9b0a-7aaf9b28c028"
-      (reference "J106") (unit 1) (value "Conn_02x02_Top_Bottom") (footprint "power_board_support:LM2596")
+      (reference "J106") (unit 1) (value "Conn_02x02_Top_Bottom") (footprint "power_board_support:LM2596-2")
     )
     (path "/f769bbb1-d71c-475e-8e96-2bf6bcda2c03"
-      (reference "J107") (unit 1) (value "Conn_02x02_Top_Bottom") (footprint "power_board_support:LM2596")
+      (reference "J107") (unit 1) (value "Conn_02x02_Top_Bottom") (footprint "power_board_support:LM2596-2")
     )
     (path "/5c31fb08-a1cc-4a5a-afba-aeb7592f39b3"
