File: boards/SIC431/SIC431/SIC431.kicad_pcb (KiCad board)
At the start: 2 copper layers, 127 x 127 mm, 82 parts, among them J101 Screw_Terminal_01x02, J102 Screw_Terminal_01x06, J103 Screw_Terminal_01x06, J104 Screw_Terminal_01x06, K101 Relay, K102 Relay, K103 Relay, K104 Relay, K105 Relay, K106 Relay, U101 SIC431AED-T1-GE3, U102 SIC431AED-T1-GE3, U103 SIC431AED-T1-GE3

Commit message: update on E-stop
Parts:
- added SW101: SW_Push_Open, power_board_support:E-Stop, F.Cu at (54.0, 39.6)
- moved K102 14.4 mm to (124.8, 89.8), turned to -90 degrees
- moved R128 8.54 mm to (119.8, 121.5), turned to 90 degrees
- moved D113 5.37 mm to (119.8, 117.7), turned to -90 degrees
- moved R130 4.10 mm to (75.5, 121.5), turned to 90 degrees
- moved D115 3.58 mm to (75.5, 117.7), turned to -90 degrees
- moved D112 1.58 mm to (114.0, 85.0)
- moved R127 1.58 mm to (118.0, 85.1)
- moved R129 0.93 mm to (99.5, 121.5), turned to 90 degrees
- moved D114 0.31 mm to (99.5, 117.7), turned to -90 degrees
Connections:
- K101 pad 1: /12V -> /V_BAT_IN
- K101 pad 2: /12V -> /E-stop
- K102 pad 1: /12V -> /V_BAT_IN
- K102 pad 2: /12V -> /E-stop
- K103 pad 1: /12V -> /V_BAT_IN
- K103 pad 2: /12V -> /E-stop
- K104 pad 1: /12V -> /V_BAT_IN
- K104 pad 2: /12V -> /E-stop
- K105 pad 1: /12V -> /V_BAT_IN
- K105 pad 2: /12V -> /E-stop
- K106 pad 1: /12V -> /V_BAT_IN
- K106 pad 2: /12V -> /E-stop
Routing:
- net /V_BAT_IN: track 17.4 -> 294.7 mm
- net /E-stop: track 0.00 -> 273.6 mm
- net /12V: track 86.6 -> 0.00 mm
- net /12V_GND_5: track 4.02 -> 23.3 mm
- net /12V_GND_4: track 4.02 -> 23.3 mm
- net /12V_GND_6: track 4.02 -> 21.8 mm
- net Net-(D102-Pad1): track 10.7 -> 21.4 mm
- net Net-(D115-Pad2): track 0.00 -> 1.87 mm
- net Net-(D114-Pad2): track 0.00 -> 1.87 mm
- net Net-(D113-Pad2): track 0.00 -> 1.86 mm
- net /12V_GND_3: track 26.7 -> 28.0 mm

Commit message: update
Parts:
- moved D107 145.8 mm to (53.5, 127.8), turned to -90 degrees
- moved D109 138.6 mm to (40.8, 127.8), turned to -90 degrees
- moved L102 104.4 mm to (-52.5, 123.5)
- moved D108 84.4 mm to (66.2, 127.8), turned to -90 degrees
- moved R117 78.8 mm to (-57.1, 104.5), turned to 180 degrees
- moved R113 56.7 mm to (-31.9, 71.5), turned to -90 degrees
- moved C101 56.5 mm to (-34.9, 66.9)
- moved R107 54.4 mm to (-25.8, 70.2), turned to 180 degrees
- moved R110 52.0 mm to (-22.9, 72.9), turned to -90 degrees
- moved L103 50.4 mm to (-87.2, 160.5)
- moved C104 49.9 mm to (-27.7, 67.1)
- moved C107 47.6 mm to (-22.9, 69.3), turned to 90 degrees
- moved C105 47.1 mm to (-52.0, 97.6)
- moved C115 46.3 mm to (-59.3, 156.6)
- moved R112 46.3 mm to (-57.1, 165.6)
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Connections:
- C101 pad 2: Earth -> GND
- C102 pad 2: Earth -> GND
- C103 pad 2: Earth -> GND
- C104 pad 2: Earth -> GND
- C105 pad 2: Earth -> GND
- C106 pad 2: Earth -> GND
- C110 pad 2: Earth -> GND
- C111 pad 2: Earth -> GND
- C112 pad 2: Earth -> GND
- C116 pad 2: Earth -> GND
- C117 pad 2: Earth -> GND
- C118 pad 2: Earth -> GND
- C119 pad 2: Earth -> GND
- C120 pad 2: Earth -> GND
- C121 pad 2: Earth -> GND
- D107 pad 1: unconnected-(D107-Pad1) -> Net-(C117-Pad1)
- D108 pad 1: unconnected-(D108-Pad1) -> Net-(C116-Pad1)
- R102 pad 2: Earth -> GND
- R104 pad 2: Earth -> GND
- R106 pad 2: Earth -> GND
- U101 pad 13: Earth -> GND
- U101 pad 27_1: Earth -> GND
- U101 pad 27_2: Earth -> GND
- U101 pad 3: Earth -> GND
- U101 pad 4: Earth -> GND
- U102 pad 13: Earth -> GND
- U102 pad 27_1: Earth -> GND
- U102 pad 27_2: Earth -> GND
- U102 pad 3: Earth -> GND
- U102 pad 4: Earth -> GND
- U103 pad 13: Earth -> GND
- U103 pad 27_1: Earth -> GND
- U103 pad 27_2: Earth -> GND
- U103 pad 3: Earth -> GND
- U103 pad 4: Earth -> GND
Routing:
- net Net-(C116-Pad1): track 0.00 -> 27.7 mm, vias 0 -> 2
- net Net-(C107-Pad1): track 0.00 -> 14.8 mm, vias 0 -> 2
- net /V_BAT_IN: track 294.7 -> 309.0 mm, vias 0 -> 2
- net Net-(L101-Pad1): track 0.00 -> 13.0 mm
- net /5V_OUT_1: track 0.00 -> 11.9 mm
- net /5V_OUT_3: track 0.00 -> 11.9 mm
- net Net-(R110-Pad2): track 0.00 -> 10.9 mm, vias 0 -> 2
- net /5V_OUT_2: track 0.00 -> 10.8 mm
- net Net-(R107-Pad2): track 0.65 -> 11.1 mm, vias 0 -> 2
- net Net-(R119-Pad1): track 0.00 -> 9.79 mm
- net Net-(R113-Pad2): track 0.00 -> 7.31 mm, vias 0 -> 2
- net Net-(R103-Pad2): track 0.00 -> 4.67 mm
- net Net-(C117-Pad1): track 0.00 -> 4.23 mm
- net Net-(C113-Pad1): track 1.80 -> 5.44 mm
- net Net-(C111-Pad1): track 0.00 -> 2.59 mm
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
Commit message: modification
Parts:
- C107, C108, R107, R108, R110, R111, R113, R114: moved to B.Cu
- moved L101 90.4 mm to (65.6, 84.2)
- moved R114 89.2 mm to (31.7, 82.6), turned to -90 degrees
- moved C102 88.7 mm to (24.1, 86.8)
- moved C105 88.7 mm to (35.0, 80.3)
- moved R103 88.3 mm to (35.1, 85.7)
- moved R104 88.3 mm to (37.4, 85.7)
- moved C114 88.0 mm to (29.2, 85.0)
- moved U102 88.0 mm to (33.0, 90.9)
- moved R117 88.0 mm to (29.1, 87.2)
- moved C111 88.0 mm to (36.8, 94.3)
- moved L102 88.0 mm to (33.8, 106.2)
- moved C108 85.1 mm to (40.8, 82.0), turned to 90 degrees
- moved R108 84.4 mm to (35.5, 84.2), turned to 180 degrees
- moved C117 84.1 mm to (41.3, 90.6)
- moved R120 84.1 mm to (39.0, 89.1)
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Routing:
- net Net-(C116-Pad1): track 27.7 -> 73.2 mm
- net /V_BAT_IN: track 309.0 -> 327.7 mm, vias 2 -> 0
- net Net-(R111-Pad2): track 0.00 -> 7.78 mm, vias 0 -> 1
- net Net-(L101-Pad1): track 13.0 -> 19.7 mm
- net Net-(R107-Pad2): track 11.1 -> 5.04 mm, vias 2 -> 1
- net Net-(L102-Pad1): track 0.00 -> 4.84 mm
- net Net-(C107-Pad1): track 14.8 -> 10.0 mm, vias 2 -> 1
- net Net-(C114-Pad1): track 0.00 -> 4.76 mm
- net Net-(R120-Pad1): track 1.66 -> 5.90 mm
- net Net-(C108-Pad1): track 0.00 -> 3.97 mm, vias 0 -> 1
- net Net-(R110-Pad2): track 10.9 -> 7.34 mm, vias 2 -> 1
- net Net-(R119-Pad1): track 9.79 -> 7.35 mm
- net Net-(R117-Pad1): track 0.00 -> 2.43 mm
- net Net-(R108-Pad2): track 0.00 -> 2.20 mm, vias 0 -> 1
- net Net-(C114-Pad2): track 0.00 -> 2.18 mm
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
Commit message: updates
Parts:
- added J105: Conn_02x02_Top_Bottom, power_board_support:LM2596, B.Cu at (32.3, 89.9)
- added J106: Conn_02x02_Top_Bottom, power_board_support:LM2596, B.Cu at (79.0, 89.9)
- added J107: Conn_02x02_Top_Bottom, power_board_support:LM2596, B.Cu at (55.5, 89.9)
- added J108: Screw_Terminal_01x02, Connector_PinHeader_2.54mm:PinHeader_1x02_P2.54mm_Vertical, F.Cu at (60.8, 134.8)
- added J109: Screw_Terminal_01x02, Connector_PinHeader_2.54mm:PinHeader_1x02_P2.54mm_Vertical, F.Cu at (48.4, 134.8)
- added J110: Screw_Terminal_01x02, Connector_PinHeader_2.54mm:PinHeader_1x02_P2.54mm_Vertical, F.Cu at (35.0, 134.8)
- added REF**: MountingHole_3mm_Pad_Via, MountingHole:MountingHole_3mm_Pad_Via, F.Cu at (8.94, 91.3)
- added REF**: MountingHole_3.5mm_Pad_Via, MountingHole:MountingHole_3.5mm_Pad_Via, F.Cu at (27.0, 27.0)
- added REF**: MountingHole_3.5mm_Pad_Via, MountingHole:MountingHole_3.5mm_Pad_Via, F.Cu at (27.0, 140.0)
- added REF**: MountingHole_3.5mm_Pad_Via, MountingHole:MountingHole_3.5mm_Pad_Via, F.Cu at (140.0, 27.0)
- added REF**: MountingHole_3.5mm_Pad_Via, MountingHole:MountingHole_3.5mm_Pad_Via, F.Cu at (140.0, 140.0)
- C101, C102, C103: footprint Capacitor_SMD:C_0805_2012Metric -> Capacitor_THT:CP_Radial_D12.5mm_P5.00mm
- C109, R109, R112, R115: moved to B.Cu
- moved C103 148.0 mm to (28.2, 59.4)
- moved C118 126.9 mm to (41.7, 98.8)
- moved L103 126.9 mm to (29.3, 110.4)
- moved R106 126.7 mm to (34.6, 90.2)
- moved R118 125.9 mm to (27.3, 92.8), turned to 180 degrees
- moved C121 122.5 mm to (38.8, 97.8), turned to 90 degrees
- moved U103 120.5 mm to (30.7, 96.5)
- moved C106 119.2 mm to (31.1, 88.1)
- moved C112 118.6 mm to (34.5, 99.7), turned to -90 degrees
- moved C109 117.4 mm to (37.7, 93.0)
- moved R112 116.9 mm to (36.8, 95.9), turned to -90 degrees
- moved R115 116.4 mm to (31.6, 96.0), turned to 90 degrees
- moved R121 116.0 mm to (36.7, 94.4), turned to 90 degrees
- moved R109 115.4 mm to (34.2, 93.0), turned to 180 degrees
- moved R124 110.5 mm to (36.7, 97.8), turned to -90 degrees
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Routing:
- net Net-(C116-Pad1): track 73.2 -> 12.1 mm
- net /V_BAT_IN: track 327.7 -> 383.1 mm
- net Net-(C117-Pad1): track 4.27 -> 32.3 mm, vias 0 -> 2
- net /12V_GND_1: track 30.1 -> 8.26 mm
- net /12V_GND_2: track 28.3 -> 8.18 mm
- net /12V_GND_3: track 28.0 -> 8.12 mm
- net /E-stop: track 273.6 -> 254.0 mm
- net Net-(C118-Pad1): track 0.00 -> 16.9 mm, vias 0 -> 2
- net Net-(L101-Pad1): track 19.7 -> 4.04 mm
- net /12V_GND_5: track 23.3 -> 8.19 mm
- net /12V_GND_4: track 23.3 -> 8.17 mm
- net /5V_OUT_3: track 11.9 -> 26.8 mm
- net /12V_GND_6: track 21.8 -> 8.15 mm
- net /5V_OUT_2: track 10.8 -> 23.6 mm
- net /5V_OUT_1: track 11.9 -> 22.7 mm
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
Commit message: mostly complete
Parts:
- removed the REF** at (8.94, 91.3)
- added G***: LOGO, Custom_Silkscreen_and_memes:IRIS_logo, F.Cu at (83.1, 49.0)
- added G***: LOGO, Custom_Silkscreen_and_memes:IRIS_OLD_logo, B.Cu at (138.1, 110.6)
- J105, J106, J107: footprint power_board_support:LM2596 -> power_board_support:LM2596-2
- moved D106 6.87 mm to (96.6, 114.6)
- moved J106 2.22 mm to (77.1, 91.2)
- moved J107 1.26 mm to (55.1, 91.1)
- moved J105 1.26 mm to (33.0, 91.0)
Routing:
- net /V_BAT_IN: track 383.1 -> 491.7 mm
- net Net-(C116-Pad1): track 12.1 -> 49.9 mm
- net Net-(C118-Pad1): track 16.9 -> 39.8 mm
- net Net-(L103-Pad1): track 2.73 -> 16.0 mm
- net Net-(C117-Pad1): track 32.3 -> 42.1 mm
- net Net-(L101-Pad1): track 4.04 -> 13.0 mm
- net Net-(L102-Pad1): track 7.33 -> 14.2 mm
- net Net-(D106-Pad1): track 7.22 -> 10.7 mm
- net /12V_IN_6: track 16.5 -> 19.0 mm
Other:
- board text added: "+"
- board text added: "-"
- board text added: "12V output"
- board text added: "5V output"
- board text added: "VBAT INPUT"
- board text added: "V_BAT_IN"

Commit message: final update, gerbers go go
final update, gerbers go go
Parts:
- moved G*** 3.52 mm to (134.6, 110.3)
Routing:
- net /GL: track 2.88 -> 6.28 mm
- net /V_BAT_IN: track 491.7 -> 492.7 mm
- net GND: vias 0 -> 59
Other:
- board text added: "Andrew Scott, Emily Lory, Buffett Lee, Joshua Meier, Nathan Colunga"
- board text added: "JLCJLCJLCJLC"
- board text added: "PROBEPCBPCB"
