File: boards/Power Distribution Board Ver.2/Power Distribution Board Ver.2.kicad_sch (KiCad schematic)
At the start: 89 parts, among them J1 Screw_Terminal_01x02, J10 Screw_Terminal_01x02, J2 Screw_Terminal_01x06, J3 Screw_Terminal_01x06, J4 Screw_Terminal_01x06, J5 Conn_02x02_Top_Bottom, J6 Conn_02x02_Top_Bottom, J7 Conn_02x02_Top_Bottom, J8 Screw_Terminal_01x02, J9 Screw_Terminal_01x02, K1 Relay, K2 Relay, K3 Relay, K4 Relay, K5 Relay, K6 Relay, SW1 SW_Push_Open, U1 SIC431AED-T1-GE3, U2 SIC431AED-T1-GE3, U3 SIC431AED-T1-GE3

Commit message: Started PCB
Parts:
- removed D10, D11, D12, D13, D14, D15: LED, LED_SMD:LED_0805_2012Metric_Pad1.15x1.40mm_HandSolder, symbol Device:LED
- removed J10, J8, J9: Screw_Terminal_01x02, Connector_PinHeader_2.54mm:PinHeader_1x02_P2.54mm_Vertical, symbol Connector:Screw_Terminal_01x02
- removed J5, J6, J7: Conn_02x02_Top_Bottom, power_board_support:LM2596-2, symbol Connector_Generic:Conn_02x02_Top_Bottom
- removed R25, R26, R27, R28, R29, R30: 100k, Resistor_SMD:R_0805_2012Metric_Pad1.20x1.40mm_HandSolder, symbol Device:R_Small_US
- added C22, C23, C24, C25, C26, C27, C28, C29, C30, C31, C32, C33, C34, C35, C36, C37, C38, C39: 47uF, Capacitor_SMD:C_0805_2012Metric, symbol Device:C
- C19, C20, C21: value 22uF -> 47uF
- R18: value 3.3 -> 0
- R22, R23, R24: value 187k -> 78.7k
- R7, R8, R9: value 50k -> 100k
Connections:
- net 5V_OUT_1: now also D7.2 (K), D9.2 (K)
- net 5V_OUT_2: no longer D7.2 (K)
- net 5V_OUT_3: no longer D9.2 (K)
- net GND: now also C22.2, C23.2, C24.2, C25.2, C26.2, C27.2, C28.2, C29.2, C30.2, C31.2, C32.2, C33.2, C34.2, C35.2, C36.2, C37.2, C38.2, C39.2
- net at C18.1, D9.1 (A), L3.2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: now also C33.1, C34.1, C35.1, C36.1, C37.1, C38.1, C39.1; no longer C21.1
- net at C17.1, C20.1, D7.1 (A)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: now also C21.1, C28.1, C29.1, C30.1, C31.1, C32.1
- net at C16.1, C19.1, D8.1 (A)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: now also C22.1, C23.1, C24.1, C25.1, C26.1, C27.1
Other:
- note removed: "Backup 5 Volt Regulators"
- note removed: "Indicators"
- moved on the sheet: C19, D8
