File: boards/Power Distribution Board Ver.2/Power Distribution Board Ver.2.kicad_pcb (KiCad board)
At the start: 4 copper layers, 127 x 127 mm, 95 parts, among them J1 Screw_Terminal_01x02, J2 Screw_Terminal_01x06, J3 Screw_Terminal_01x06, J4 Screw_Terminal_01x06, K1 Relay, K2 Relay, K3 Relay, K4 Relay, K5 Relay, K6 Relay, SW1 SW_Push_Open, U1 SIC431AED-T1-GE3, U2 SIC431AED-T1-GE3, U3 SIC431AED-T1-GE3

Commit message: Aesthetics
Parts:
- moved J2 1.68 mm to (126.2, 36.3)
- moved J4 0.79 mm to (53.8, 140.5)
Routing:
- net /12V_IN_3: track 18.9 -> 17.5 mm
- net /12V_IN_2: track 19.3 -> 17.9 mm
- net /12V_IN_1: track 18.9 -> 17.5 mm
- net /5V_OUT_3: track 14.6 -> 13.8 mm
Other:
- board text added: "+"
- board text added: "12V Output"
- board text added: "5V Output"
- board text added: "IRIS - XV PROBEPCBPCB Ver. 2 Buffett Lee, Emily Lory, Joseph Hanger, Henry Lin Nathan Colunga, Ben Saarva, Jakub Wojdyla"
- board text removed: "Buffett Lee, Emily Lory, Joseph Hanger, Henry Lin, Ben Saarva, Jakub Wojdyla, Wyatt Sturn, Miaomiao Jin"

Commit message: Aesthetics
Other:
- board text added: "IRIS - XV PROBEPCBPCB Ver. 2 Buffett Lee, Emily Lory, Joseph Hanger, Henry Lin Nathan Colunga, Ben Saarva, Jakub Wojdyla Wyatt Sturn, Miaomiao Jin"
- board text removed: "IRIS - XV PROBEPCBPCB Ver. 2 Buffett Lee, Emily Lory, Joseph Hanger, Henry Lin Nathan Colunga, Ben Saarva, Jakub Wojdyla"

Commit message: Add JLC
Other:
- board text added: "JLCJLCJLCJLC"
Changed lines of the file:
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@@
+    (effects (font (size 1.5 1.5) (thickness 0.3) bold) (justify left bottom mirror))
+  )
+  (gr_text "JLCJLCJLCJLC" (at 132.588 145.034) (layer "B.SilkS")
     (effects (font (size 1.5 1.5) (thickness 0.3) bold) (justify left bottom mirror))
   )
