File: boards/Arduino Shield v2 ethernet/Arduino Shield.kicad_pcb (KiCad board)
At the start: 2 copper layers, 114.3 x 76.2 mm, 21 parts, among them J1 Screw_Terminal_01x07, J11 Screw_Terminal_01x08, J2 Screw_Terminal_01x08, J3 Screw_Terminal_01x08, J4 Screw_Terminal_01x08, J5 Screw_Terminal_01x08, J6 Screw_Terminal_01x08, J7 Screw_Terminal_01x08, J8 Screw_Terminal_01x07, J9 Screw_Terminal_01x10, U1 A000062

Commit message: finished shield v1
Parts:
- moved D4 15.2 mm to (185.2, 86.4)
- moved R1 15.2 mm to (192.1, 86.4)
- moved D2 10.2 mm to (186.4, 66.0)
- moved D1 10.2 mm to (185.4, 76.2)
- moved R3 10.2 mm to (192.1, 66.0)
- moved R5 10.2 mm to (192.1, 76.2)
- moved D3 5.09 mm to (185.2, 71.1)
- moved R2 5.08 mm to (192.1, 71.1)
- renumbered D5 to D1, D3 to D2, D1 to D3, D2 to D4, D4 to D5
Routing:
- net Net-(U1-D51): track 23.5 -> 46.7 mm
- net Net-(U1-D50): track 23.4 -> 12.7 mm, vias 0 -> 1
- net Net-(J9-Pin_2): track 18.5 -> 28.6 mm, vias 0 -> 1
- net Net-(U1-D49): track 29.6 -> 36.2 mm
- net Net-(U1-D53): track 18.9 -> 22.5 mm
- net Net-(J4-Pin_3): track 81.5 -> 84.4 mm
- net Net-(J9-Pin_4): track 16.6 -> 18.1 mm
- net Net-(J4-Pin_2): track 80.9 -> 82.4 mm
- net Net-(J4-Pin_6): track 58.5 -> 59.7 mm
- net Net-(J1-Pin_7): track 20.3 -> 21.3 mm
- net Net-(D2-A): track 4.86 -> 3.92 mm
- net Net-(J9-Pin_1): track 20.4 -> 21.1 mm
- net Net-(U1-D52): track 16.6 -> 15.9 mm
- net GND: track 0.00 -> 0.69 mm
- net Net-(D3-A): track 5.77 -> 5.10 mm
