File: boards/Arduino Shield V2 REAL/Arduino Shield.kicad_sch (KiCad schematic)
At the start: 2 parts, among them U1 W5500, U2 A000062

Commit message: E
Parts:
- removed U1: W5500, Package_QFP:LQFP-48_7x7mm_P0.5mm, symbol Interface_Ethernet:W5500
- removed U2: A000062, Arduino_Due_Shield:Arduino_Due_Shield, symbol A000062:A000062
- added ACT0, UNK100M1: Green, Arduino-Ethernet-Shield2-V2:CHIPLED_0805, symbol Arduino-Ethernet-Shield2-V2-eagle-import:0043_KPT-2012SGC
- added C1, C3: 22uF, symbol Device:C_Polarized_Small
- added C10: 4u7, symbol Device:C_Polarized_Small
- added C11: 10n, symbol Device:C_Small
- added C17, C37, C38, C44: 22uF, Arduino-Ethernet-Shield2-V2:SMC_B, symbol Arduino-Ethernet-Shield2-V2-eagle-import:0167_
- added C18, C31, C39, C40, C41, C42, C43, C45: 100n, Arduino-Ethernet-Shield2-V2:C0603-ROUND, symbol Arduino-Ethernet-Shield2-V2-eagle-import:0015_100NF_0603
- added C19, C20, C21, C26, C29, C36: 10n, Arduino-Ethernet-Shield2-V2:C0603-ROUND, symbol Arduino-Ethernet-Shield2-V2-eagle-import:0142_10NF_0603
- added C2, C4, C5, C6, C7, C8, C9: 100n, symbol Device:C_Small
- added C27, C28: 10nF, Arduino-Ethernet-Shield2-V2:C0603-ROUND, symbol Arduino-Ethernet-Shield2-V2-eagle-import:0142_10NF_0603
- added C3, C7: 10p, Arduino-Ethernet-Shield2-V2:C0603-ROUND, symbol Arduino-Ethernet-Shield2-V2-eagle-import:0245_0603C0G10PF50V
- added C46: 4u7, Arduino-Ethernet-Shield2-V2:SMC_A, symbol Arduino-Ethernet-Shield2-V2-eagle-import:0474_TAJA475M016RNJ
- added D1, D2, D3, D4, D5: LED, LED_SMD:LED_0805_2012Metric, symbol Device:LED
- added FDX1, LINK1: Yellow, Arduino-Ethernet-Shield2-V2:CHIPLED_0805, symbol Arduino-Ethernet-Shield2-V2-eagle-import:0044_KPT-2012YC
- added IC6: 0982_W5500, Arduino-Ethernet-Shield2-V2:TQFP48-7X7, symbol Arduino-Ethernet-Shield2-V2-eagle-import:0982_W5500
- added J1, J8: Screw_Terminal_01x07, TerminalBlock_4Ucon:TerminalBlock_4Ucon_1x07_P3.50mm_Horizontal, symbol Connector:Screw_Terminal_01x07
- added J11, J2, J3, J4, J5, J6, J7: Screw_Terminal_01x08, TerminalBlock_4Ucon:TerminalBlock_4Ucon_1x08_P3.50mm_Horizontal, symbol Connector:Screw_Terminal_01x08
- added J9: Screw_Terminal_01x10, TerminalBlock_4Ucon:TerminalBlock_4Ucon_1x10_P3.50mm_Horizontal, symbol Connector:Screw_Terminal_01x10
- added L12, L2: MH2029-300Y, Arduino-Ethernet-Shield2-V2:0805, symbol Arduino-Ethernet-Shield2-V2-eagle-import:0001_BLM21PG300SN1D_/_MH2029-300Y
- added Q2: 25MHz KX-7_NM, Arduino-Ethernet-Shield2-V2:CRYSTAL3.2X2.5, symbol Arduino-Ethernet-Shield2-V2-eagle-import:0846_FTX25.000M12SM3S
- added R1, R2, R3, R5: 6Ω, Resistor_SMD:R_0805_2012Metric, symbol Device:R_Small_US
- added R10, R11, R12, R15, R20, R9: 10k, Arduino-Ethernet-Shield2-V2:R0603-ROUND, symbol Arduino-Ethernet-Shield2-V2-eagle-import:0028_CR0603JW103L
- added R13, R21: 0R, Arduino-Ethernet-Shield2-V2:R0402, symbol Arduino-Ethernet-Shield2-V2-eagle-import:0039_JUMP_0402
- added R22, R23: 10k, Arduino-Ethernet-Shield2-V2:R0603-ROUND, symbol Arduino-Ethernet-Shield2-V2-eagle-import:0131_CR0603FX1000L
- added R24: 22R, Arduino-Ethernet-Shield2-V2:R0603-ROUND, symbol Arduino-Ethernet-Shield2-V2-eagle-import:0247_22R_0603
- added R3: 1M, Arduino-Ethernet-Shield2-V2:R0603-ROUND, symbol Arduino-Ethernet-Shield2-V2-eagle-import:0004_0603_1M
- added R4: 10K, Arduino-Ethernet-Shield2-V2:R0603-ROUND, symbol Arduino-Ethernet-Shield2-V2-eagle-import:0028_CR0603JW103L
- added R4: 232Ω, Resistor_SMD:R_0805_2012Metric, symbol Device:R_Small_US
- added R8: 12k4_1%, Arduino-Ethernet-Shield2-V2:R0603-ROUND, symbol Arduino-Ethernet-Shield2-V2-eagle-import:0984_12K4_1%_0603
- added RN11: 49R9, Arduino-Ethernet-Shield2-V2:CAY16, symbol Arduino-Ethernet-Shield2-V2-eagle-import:0036_CAY16-49R9F4L
- added RN3: 470R, Arduino-Ethernet-Shield2-V2:CAY16, symbol Arduino-Ethernet-Shield2-V2-eagle-import:0540_CAY16-471J4LF
- added RN8, RN9: 10k, Arduino-Ethernet-Shield2-V2:CAY16, symbol Arduino-Ethernet-Shield2-V2-eagle-import:0016_064R_10K_/_CAY16-103J4LF
- added T2: PMV48XP, Arduino-Ethernet-Shield2-V2:SOT-23, symbol Arduino-Ethernet-Shield2-V2-eagle-import:0297_PMV48XP
- added U1: A000062, Arduino_Due_Shield:Arduino_Due_Shield, symbol A000062:A000062
- added U2: W5500, Package_QFP:LQFP-48_7x7mm_P0.5mm, symbol Interface_Ethernet:W5500
- added UC1: RB1-125BHQ1A, Arduino-Ethernet-Shield2-V2:POE-RJ45, symbol Arduino-Ethernet-Shield2-V2-eagle-import:0033_RB1-125BHQ1A
Connections:
- new net: C3.2, C5.2, U2.29 (GND)
- new net: LINK1.A, RN3.6 (2), UC1.L3 (L3G+)
- new net: J3.1 (Pin_1), U1.CANTX0
- new net: J3.2 (Pin_2), U1.CANRX0
- new net: J3.3 (Pin_3), U1.DAC1
- new net: J3.4 (Pin_4), U1.DAC0
- new net: J3.5 (Pin_5), U1.AD11 (ADC11)
- new net: J3.6 (Pin_6), U1.AD10 (ADC10)
- new net: J3.7 (Pin_7), U1.AD9 (ADC9)
- new net: J3.8 (Pin_8), U1.AD8 (ADC8)
- new net: J2.1 (Pin_1), U1.AD7 (ADC7)
- new net: J2.2 (Pin_2), U1.AD6 (ADC6)
- new net: J2.3 (Pin_3), U1.AD5 (ADC5)
- new net: J2.4 (Pin_4), U1.AD4 (ADC4)
- new net: J2.5 (Pin_5), U1.AD3 (ADC3)
- new net: J2.6 (Pin_6), U1.AD2 (ADC2)
- new net: J2.7 (Pin_7), U1.AD1 (ADC1)
- new net: J2.8 (Pin_8), U1.AD0 (ADC0)
- new net: C3.1, IC6.31 (XO), Q2.1, R3.1
- new net: D5.2 (A), R5.1
- new net: R5.2, U1.53 (D53)
- new net: IC6.42 (RSVD5), RN9.1
- new net: IC6.23 (RSVD), R4.2
- new net: J9.1 (Pin_1), U1.SCL
- new net: J9.10 (Pin_10), U1.8 (D8)
- new net: J9.2 (Pin_2), U1.SDA
- new net: J9.3 (Pin_3), U1.AREF
- new net: J9.5 (Pin_5), U1.13 (D13)
- new net: J9.6 (Pin_6), U1.12 (D12)
- new net: J9.7 (Pin_7), U1.11 (D11)
- new net: J9.8 (Pin_8), U1.10 (D10)
- new net: J9.9 (Pin_9), U1.9 (D9)
- new net: J1.1 (Pin_1), U1.VIN
- new net: J1.4 (Pin_4), U1.5V_1 (+5V_1)
- new net: J1.5 (Pin_5), U1.3V3 (+3V3)
- new net: J1.6 (Pin_6), U1.RESET (~{RESET})
- new net: J1.7 (Pin_7), U1.IOREF
- new net: C28.2, UC1.R2 (RD-)
- new net: J4.1 (Pin_1), U1.34 (D34)
- new net: J4.2 (Pin_2), U1.32 (D32)
- new net: J4.3 (Pin_3), U1.30 (D30)
- new net: J4.4 (Pin_4), U1.28 (D28)
- new net: J4.5 (Pin_5), U1.26 (D26)
- new net: J4.6 (Pin_6), U1.24 (D24)
- new net: J4.7 (Pin_7), U1.22 (D22)
- new net: J4.8 (Pin_8), U1.5V_2 (+5V_2)
- new net: IC6.10 (EXRES1), R8.2
- new net: C46.+, IC6.20 (TOCAP)
- new net: C7.1, IC6.30 (XI/CLKIN), Q2.3, R3.2
- new net: IC6.38 (RSVD1), RN8.1
- new net: IC6.39 (RSVD2), RN9.4 (1)
- new net: IC6.40 (RSVD3), RN9.3 (1)
- new net: IC6.41 (RSVD4), RN9.2 (1)
- new net: J5.1 (Pin_1), U1.7 (D7)
- new net: J5.2 (Pin_2), U1.6 (D6)
- new net: J5.3 (Pin_3), U1.5 (D5)
- new net: J5.4 (Pin_4), U1.4 (D4)
- new net: J5.5 (Pin_5), U1.3 (D3)
- new net: J5.6 (Pin_6), U1.2 (D2)
- new net: J5.7 (Pin_7), U1.1 (D1/TX0)
- new net: J5.8 (Pin_8), U1.0 (D0/RX0)
- new net: C11.1, U2.22 (1V2O)
- new net: D4.2 (A), R4.1
- new net: R4.2, U1.52 (D52)
- new net: D1.2 (A), R2.1
- new net: R2.2, U1.49 (D49)
- new net: FDX1.A, RN3.7 (2)
- new net: Q2.2, R13.2
- new net: Q2.4, R21.1
- new net: D3.2 (A), R3.1
- new net: R3.2, U1.51 (D51)
- new net: C19.2, R22.1, R23.1
- new net: D2.2 (A), R1.1
- new net: R1.2, U1.50 (D50)
- new net: ACT0.A, RN3.8 (2)
- new net: C31.2, R24.2, UC1.R3 (CT)
- new net: RN3.5 (2), UC1.L1 (L1Y+), UNK100M1.A
- new net: C27.2, UC1.R1 (RD+)
- new net: C10.1, U2.20 (TOCAP)
- new net: J7.1 (Pin_1), U1.5V_3 (+5V_3)
- new net: J7.2 (Pin_2), U1.23 (D23)
- new net: J7.3 (Pin_3), U1.25 (D25)
- new net: J7.4 (Pin_4), U1.27 (D27)
- new net: J7.5 (Pin_5), U1.29 (D29)
- new net: J7.6 (Pin_6), U1.31 (D31)
- new net: J7.7 (Pin_7), U1.33 (D33)
- new net: J7.8 (Pin_8), U1.35 (D35)
- new net: J6.1 (Pin_1), U1.14 (D14/TX3)
- new net: J6.2 (Pin_2), U1.15 (D15/RX3)
- new net: J6.3 (Pin_3), U1.16 (D16/TX2)
- new net: J6.4 (Pin_4), U1.17 (D17/RX2)
- new net: J6.5 (Pin_5), U1.18 (D18/TX1)
- new net: J6.6 (Pin_6), U1.19 (D19/RX1)
- new net: J6.7 (Pin_7), U1.20 (D20/SDA)
- new net: J6.8 (Pin_8), U1.21 (D21/SCL)
- new net: J11.8 (Pin_8), U1.36 (D36)
- new net: J8.1 (Pin_1), U1.37 (D37)
- new net: J11.7 (Pin_7), U1.38 (D38)
- new net: J8.2 (Pin_2), U1.39 (D39)
- new net: J11.6 (Pin_6), U1.40 (D40)
- new net: J8.3 (Pin_3), U1.41 (D41)
- new net: J11.5 (Pin_5), U1.42 (D42)
- new net: J8.4 (Pin_4), U1.43 (D43)
- new net: J11.4 (Pin_4), U1.44 (D44)
- new net: J8.5 (Pin_5), U1.45 (D45)
- new net: J11.3 (Pin_3), U1.46 (D46)
- new net: J8.6 (Pin_6), U1.47 (D47)
- new net: J11.2 (Pin_2), U1.48 (D48)
- new net +3V3: C1.1, C2.2, C3.1, C4.2, C5.1, C6.2, C7.2, C8.2, C9.2, L12.1, L2.1, T2.2 (S), U2.11 (AVDD), U2.15 (AVDD), U2.17 (AVDD), U2.21 (AVDD), U2.28 (VDD), U2.4 (AVDD), U2.8 (AVDD)
- new net +3V3A: C38.+, C39.1, C40.1, C41.1, C42.1, C43.1, C44.+, C45.1, IC6.11 (AVDD2), IC6.15 (AVDD3), IC6.17 (AVDD4), IC6.21 (AVDD5), IC6.4 (AVDD), IC6.8 (AVDD1), L12.2, R24.1, RN11.1, RN11.2 (1)
- new net +3V3D: C17.+, C18.2, C37.+, IC6.28 (VDD), L2.2, R10.2, R12.2, R9.2, RN8.5 (2), RN8.6 (2), RN8.7 (2)
- new net 1V2O: C36.2, IC6.22 (1V2O)
- new net 3V3_LED: RN3.1, RN3.2 (1), RN3.3 (1), RN3.4 (1), T2.1 (D)
- new net ACT: ACT0.C, IC6.27 (ACTLED)
- new net FDXLED: FDX1.C, IC6.26 (DUPLED)
- new net GND: C1.2, C10.2, C11.2, C17.-, C18.1, C19.1, C2.1, C20.1, C21.1, C26.1, C29.1, C3.2, C31.1, C36.1, C37.-, C38.-, C39.2, C4.1, C40.2, C41.2, C42.2, C43.2, C44.-, C45.2, C46.-, C6.1, C7.1, C7.2, C8.1, C9.1, D1.1 (K), D2.1 (K), D3.1 (K), D4.1 (K), D5.1 (K), IC6.14 (AGND2), IC6.16 (AGND3), IC6.19 (AGND4), IC6.29 (GND), IC6.3 (AGND), IC6.48 (AGND5), IC6.9 (AGND1), J1.2 (Pin_2), J1.3 (Pin_3), J11.1 (Pin_1), J8.7 (Pin_7), J9.4 (Pin_4), R11.1, R13.1, R15.1, R20.1, R21.2, R4.1, R8.1, RN8.8 (2), RN9.5 (2), RN9.6 (2), RN9.7 (2), RN9.8 (2), U1.GND1, U1.GND2, U1.GND3, U1.GND4, U1.GND5, U2.14 (AGND), U2.16 (AGND), U2.19 (AGND), U2.3 (AGND), U2.48 (AGND), U2.9 (AGND), UC1.CH1, UC1.CH2
- new net INT: IC6.36 (INTN), RN8.4 (1)
- new net IO10*/SS: IC6.32 (SCSN), RN8.3 (1)
- new net LINKLED: IC6.25 (LINKLED), LINK1.C, T2.3 (G), UC1.L4 (L4G-)
- new net MISO: IC6.34 (MISO)
- new net MOSI3: IC6.35 (MOSI)
- new net NC: IC6.12 (NC)
- new net PMODE0: IC6.45 (PMODE0), R11.2, R9.1
- new net PMODE1: IC6.44 (PMODE1), R12.1, R15.2
- new net PMODE2: IC6.43 (PMODE2), R10.1, R20.2
- new net RESET_W: IC6.37 (RSTN), RN8.2 (1)
- new net RXIN: C28.1, IC6.5 (RXN), R22.2
- new net RXIP: C27.1, IC6.6 (RXP), R23.2
- new net SCK3: IC6.33 (SCLK)
- new net SPDLED: IC6.24 (SPDLED), UC1.L2 (L2Y-), UNK100M1.C
- new net TXON: IC6.1 (TXN), RN11.7 (2), UC1.R4 (TD-)
- new net TXOP: IC6.2 (TXP), RN11.8 (2), UC1.R5 (TD+)
- new net V1+: C20.2, UC1.R10 (SPARE2)
- new net V1-: C21.2, UC1.R9 (SPARE1)
- new net V2+: C29.2, UC1.R7 (RXCT)
- new net V2-: C26.2, UC1.R8 (TXCT)
Other:
- note added: "ETH-POE"
- note added: "NON MONTARE R11, R15, R20 ALL CAPATIBLE, AUTO NEGOTIATION ENABLE"
