File: boards/Arduino Shield V2 REAL/Arduino Shield.kicad_sch (KiCad schematic)
At the start: 84 parts, among them IC6 0982_W5500, J1 Screw_Terminal_01x07, J11 Screw_Terminal_01x08, J2 Screw_Terminal_01x08, J3 Screw_Terminal_01x08, J4 Screw_Terminal_01x08, J5 Screw_Terminal_01x08, J6 Screw_Terminal_01x08, J7 Screw_Terminal_01x08, J8 Screw_Terminal_01x07, J9 Screw_Terminal_01x10, Q2 25MHz KX-7_NM, T2 PMV48XP, U1 A000062, U2 W5500

Commit message: Updated Arduino Shield V2 ethernet schematic
Parts:
- added D6, D7: LED, LED_SMD:LED_0805_2012Metric, symbol Device:LED
- added J10: RJ45_Abracon_ARJP11A-MASA-B-A-EMU2, Connector_RJ:RJ45_Abracon_ARJP11A-MA_Horizontal, symbol Connector:RJ45_Abracon_ARJP11A-MASA-B-A-EMU2
- added R20, R24, R25, R26, R27, R28, R29, R30, R31, R32, R33, R34, R35, R36, R37: 10kΩ, Resistor_SMD:R_0805_2012Metric, symbol Device:R_Small_US
- added R21: 12k4Ω, Resistor_SMD:R_0805_2012Metric, symbol Device:R_Small_US
- added R22, R23: 470Ω, Resistor_SMD:R_0805_2012Metric, symbol Device:R_Small_US
- added T2: PMV48XP, Arduino-Ethernet-Shield2-V2:SOT-23, symbol Arduino-Ethernet-Shield2-V2-eagle-import:0297_PMV48XP
Connections:
- net +3V3: now also R29.2, R30.2, R33.1, R35.1, R37.1, T2.2 (S)
- net ACT: now also U2.27 (ACTLED), D7.1 (K)
- net FDXLED: now also U2.26 (DUPLED), D6.1 (K)
- net GND: now also R20.2, R21.2, R24.2, R25.2, R26.2, R27.2, R28.2, R32.2, R34.2, R36.2
- net LINKLED: now also U2.25 (LINKLED), T2.3 (G)
- net MISO: now also U2.34 (MISO)
- net MOSI3: now also U2.35 (MOSI)
- net PMODE0: now also U2.43 (PMODE2), R35.2, R36.1
- net PMODE1: now also U2.44 (PMODE1), R33.2, R34.1
- net PMODE2: now also U2.45 (PMODE0), R32.1, R37.2
- net RESET_W: now also U2.37 (~{RST})
- net RXIN: now also U2.5 (RXN)
- net RXIP: now also U2.6 (RXP)
- net SCK3: now also U2.33 (SCLK)
- net SPDLED: now also U2.24 (SPDLED)
- net TXON: now also U2.1 (TXN)
- net TXOP: now also U2.2 (TXP)
- net at U2.10 (EXRES1): now also R21.1
- net at U2.23 (RSVD): now also R20.1
- net at U2.32 (~{SCS}): now also R29.1
- net at U2.36 (~{INT}): now also R30.1
- net at U2.38 (RSVD): now also R28.1
- net at U2.39 (RSVD): now also R24.1
- net at U2.40 (RSVD): now also R25.1
- net at U2.41 (RSVD): now also R26.1
- net at U2.42 (RSVD): now also R27.1
- new net: R22.2, R23.1, T2.1 (D)
- new net: D7.2 (A), R23.2
- new net: D6.2 (A), R22.1
Other:
- moved on the sheet: ACT0, C17, C18, C3, C36, C37, C38, C39, C40, C41, C42, C43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

Commit message: Updated schematic for ethernet shield
Parts:
- added C35, C36: 10p, symbol Device:C_Small
- added Q2: 25MHz KX-7_NM, Arduino-Ethernet-Shield2-V2:CRYSTAL3.2X2.5, symbol Arduino-Ethernet-Shield2-V2-eagle-import:0846_FTX25.000M12SM3S
- added R38, R39: 0R, Resistor_SMD:R_0805_2012Metric, symbol Device:R_Small_US
- added R40: 1MΩ, Resistor_SMD:R_0805_2012Metric, symbol Device:R_Small_US
Connections:
- net GND: now also C35.1, C36.1, R38.1, R39.2
- net at U2.30 (XI/CLKIN): now also C36.2, Q2.3, R40.2
- net at U2.31 (XO): now also C35.2, Q2.1, R40.1
- new net: Q2.2, R39.1
- new net: Q2.4, R38.2
Other:
- moved on the sheet: ACT0, C17, C18, C3, C36, C37, C38, C39, C40, C41, C42, C43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

Commit message: Finished wiring POE and W5500 on schematic
Parts:
- removed ACT0, UNK100M1: Green, Arduino-Ethernet-Shield2-V2:CHIPLED_0805, symbol Arduino-Ethernet-Shield2-V2-eagle-import:0043_KPT-2012SGC
- removed C17, C37, C38, C44: 22uF, Arduino-Ethernet-Shield2-V2:SMC_B, symbol Arduino-Ethernet-Shield2-V2-eagle-import:0167_
- removed C18, C31, C39, C40, C41, C42, C43, C45: 100n, Arduino-Ethernet-Shield2-V2:C0603-ROUND, symbol Arduino-Ethernet-Shield2-V2-eagle-import:0015_100NF_0603
- removed C19, C20, C21, C26, C29, C36: 10n, Arduino-Ethernet-Shield2-V2:C0603-ROUND, symbol Arduino-Ethernet-Shield2-V2-eagle-import:0142_10NF_0603
- removed C27, C28: 10nF, Arduino-Ethernet-Shield2-V2:C0603-ROUND, symbol Arduino-Ethernet-Shield2-V2-eagle-import:0142_10NF_0603
- removed C3, C7: 10p, Arduino-Ethernet-Shield2-V2:C0603-ROUND, symbol Arduino-Ethernet-Shield2-V2-eagle-import:0245_0603C0G10PF50V
- removed C46: 4u7, Arduino-Ethernet-Shield2-V2:SMC_A, symbol Arduino-Ethernet-Shield2-V2-eagle-import:0474_TAJA475M016RNJ
- removed FDX1, LINK1: Yellow, Arduino-Ethernet-Shield2-V2:CHIPLED_0805, symbol Arduino-Ethernet-Shield2-V2-eagle-import:0044_KPT-2012YC
- removed IC6: 0982_W5500, Arduino-Ethernet-Shield2-V2:TQFP48-7X7, symbol Arduino-Ethernet-Shield2-V2-eagle-import:0982_W5500
- removed Q2: 25MHz KX-7_NM, Arduino-Ethernet-Shield2-V2:CRYSTAL3.2X2.5, symbol Arduino-Ethernet-Shield2-V2-eagle-import:0846_FTX25.000M12SM3S
- removed R10, R11, R12, R15, R20, R9: 10k, Arduino-Ethernet-Shield2-V2:R0603-ROUND, symbol Arduino-Ethernet-Shield2-V2-eagle-import:0028_CR0603JW103L
- removed R13, R21: 0R, Arduino-Ethernet-Shield2-V2:R0402, symbol Arduino-Ethernet-Shield2-V2-eagle-import:0039_JUMP_0402
- removed R22, R23: 10k, Arduino-Ethernet-Shield2-V2:R0603-ROUND, symbol Arduino-Ethernet-Shield2-V2-eagle-import:0131_CR0603FX1000L
- removed R24: 22R, Arduino-Ethernet-Shield2-V2:R0603-ROUND, symbol Arduino-Ethernet-Shield2-V2-eagle-import:0247_22R_0603
- removed R3: 1M, Arduino-Ethernet-Shield2-V2:R0603-ROUND, symbol Arduino-Ethernet-Shield2-V2-eagle-import:0004_0603_1M
- removed R4: 10K, Arduino-Ethernet-Shield2-V2:R0603-ROUND, symbol Arduino-Ethernet-Shield2-V2-eagle-import:0028_CR0603JW103L
- removed R8: 12k4_1%, Arduino-Ethernet-Shield2-V2:R0603-ROUND, symbol Arduino-Ethernet-Shield2-V2-eagle-import:0984_12K4_1%_0603
- removed RN3: 470R, Arduino-Ethernet-Shield2-V2:CAY16, symbol Arduino-Ethernet-Shield2-V2-eagle-import:0540_CAY16-471J4LF
- removed RN8, RN9: 10k, Arduino-Ethernet-Shield2-V2:CAY16, symbol Arduino-Ethernet-Shield2-V2-eagle-import:0016_064R_10K_/_CAY16-103J4LF
- removed T2: PMV48XP, Arduino-Ethernet-Shield2-V2:SOT-23, symbol Arduino-Ethernet-Shield2-V2-eagle-import:0297_PMV48XP
- removed UC1: RB1-125BHQ1A, Arduino-Ethernet-Shield2-V2:POE-RJ45, symbol Arduino-Ethernet-Shield2-V2-eagle-import:0033_RB1-125BHQ1A
- added C12, C13, C14, C15, C16, C17, C44: 100n, symbol Device:C_Small
- added C18, C19: 22uF, symbol Device:C_Polarized_Small
- added C37, C38, C39, C40, C41, C42, C43: 10n, symbol Device:C_Small
- added D8, D9: LED, LED_SMD:LED_0805_2012Metric, symbol Device:LED
- added R41, R42: 470Ω, Resistor_SMD:R_0805_2012Metric, symbol Device:R_Small_US
- added R43, R44: 10kΩ, Resistor_SMD:R_0805_2012Metric, symbol Device:R_Small_US
- added R45: 22Ω, Resistor_SMD:R_0805_2012Metric, symbol Device:R_Small_US
Connections:
- net LINKLED is gone; now on an unnamed net: T2.3 (G), U2.25 (LINKLED)
- net SPDLED is gone; now on an unnamed net: U2.24 (SPDLED)
- net TXON is gone; now on an unnamed net: RN11.7 (2), U2.1 (TXN)
- net TXOP is gone; now on an unnamed net: RN11.8 (2), U2.2 (TXP)
- net +3V3: no longer C3.1, C5.1, U2.28 (VDD)
- net +3V3A: now also C3.1, C5.1, U2.28 (VDD), C18.1; no longer RN11.1, RN11.2 (1)
- net +3V3D: now also C19.1
- net GND: now also J10.SH, C12.2, C13.2, C14.2, C15.2, C16.2, C17.2, C18.2, C19.2, C37.1, C38.1, C39.1, C40.1, C42.2, C44.1
- net at J10.10 (V-): now also C40.2
- net at J10.11: now also D9.1 (K), R42.2
- net at J10.12: now also D9.2 (A)
- net at J10.13: now also D8.1 (K), R41.2
- net at J10.14: now also D8.2 (A)
- net at J10.3 (RD+): now also C41.2
- net at J10.4 (TCT): now also C37.2
- net at J10.5 (RCT): now also C38.2
- net at J10.6 (RD-): now also C43.2
- net at J10.7: now also C44.2, R45.1
- net at J10.9 (V+): now also C39.2
- net PMODE0: no longer names the net of R35.2, R36.1, U2.43 (PMODE2)
- net PMODE1: no longer names the net of R33.2, R34.1, U2.44 (PMODE1)
- net PMODE2: no longer names the net of R32.1, R37.2, U2.45 (PMODE0)
- net RESET_W: no longer names the net of U2.37 (~{RST})
- net RXIN: no longer names the net of U2.5 (RXN)
- net RXIN: now also C43.1, R44.1
- net RXIP: no longer names the net of U2.6 (RXP)
- net RXIP: now also C41.1, R43.2
- new net: R45.2, RN11.1, RN11.2 (1)
- new net: C42.1, R43.1, R44.2
- new net: R41.1, R42.1
- new net +5V: C12.1, C13.1, C14.1, C15.1, C16.1, C17.1
Other:
- note removed: "ETH-POE"
- note removed: "NON MONTARE R11, R15, R20 ALL CAPATIBLE, AUTO NEGOTIATION ENABLE"
