File: boards/Battery Management System/bms/bms.kicad_sch (KiCad schematic)
At the start: 25 parts, among them J1 Screw_Terminal_01x05, J2 1986660-2, J3 1986660-2, K1 HE1AN-W-DC6V-Y6, U1 BD48L32G, U2 BD48L32G, U3 BD48L32G, U4 BD48L32G, U5 Opamp_Quad, U6 74AUC2G08

Commit message: Edited schematic and PCB
Parts:
- removed R1: 5kΩ, Resistor_SMD:R_0805_2012Metric, symbol Device:R_Small_US
- removed R1: 10kΩ, Resistor_SMD:R_0805_2012Metric, symbol Device:R_Small_US
- removed U5: Opamp_Quad, footprints:SOT23_DBV_5_TEX-L, symbol Device:Opamp_Quad
- removed U6: 74AUC2G08, footprints:D14-L, symbol 74xGxx:74AUC2G08
- added R1: 10kΩ, Resistor_SMD:R_0805_2012Metric, symbol Device:R_Small_US
- added R1: 5kΩ, Resistor_SMD:R_0805_2012Metric, symbol Device:R_Small_US
- added U5: SN74HC08DR, SN74HC08DR:SOIC127P600X175-14N, symbol SN74HC08DR:SN74HC08DR
- added U6: TL071HIDBVR, TL071HIDBVR:SOT23_DBV_5_TEX-L, symbol TL071HIDBVR:TL071HIDBVR
- K1: footprint footprints:HE1AN-W-DC6V_PAN -> HE1AN_W_DC6V_Y6:HE1AN-W-DC6V_PAN
Connections:
- net CON_1: now also U5.1 (1A)
- net CON_2: now also U5.2 (1B)
- net CON_3: now also U5.4 (2A)
- net CON_4: now also U5.5 (2B)
- net GND: now also R1.1, U5.7 (GND), U6.2 (V-)
- net V_BAT_IN: now also U5.14 (VCC), U6.5 (V+)
- net at K1.5: now also R1.2, U6.1 (OUT)
- new net: U5.8 (3Y), U6.3 (IN+)
- new net: R1.1, R1.2, U6.4 (IN-)
- new net: U5.10 (3B), U5.6 (2Y)
- new net: U5.3 (1Y), U5.9 (3A)
Other:
- moved on the sheet: D1, D2, D3, D4, K1, R1

Commit message: Updated Schematic and PCB
Connections:
- net CON_1: now also U5.5 (2B); no longer U5.1 (1A)
- net CON_2: now also U5.4 (2A); no longer U5.2 (1B)
- net CON_3: now also U5.2 (1B); no longer U5.4 (2A)
- net CON_4: now also U5.1 (1A); no longer U5.5 (2B)
- net at U5.10 (3B): now also U5.3 (1Y); no longer U5.6 (2Y)
- net at U5.9 (3A): now also U5.6 (2Y); no longer U5.3 (1Y)
Changed lines of the file:
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@@
+    (stroke (width 0) (type default))
+  )
+  (wire (pts (xy 68.58 121.92) (xy 71.12 121.92))
     (stroke (width 0) (type default))
   )
@@
     (stroke (width 0) (type default))
   )
+  (wire (pts (xy 57.15 106.68) (xy 57.15 134.62))
+    (stroke (width 0) (type default))
+  )
   (wire (pts (xy 111.506 40.64) (xy 105.156 40.64))
     (stroke (width 0) (type default))
@@
     (stroke (width 0) (type default))
   )
-  (wire (pts (xy 54.61 104.14) (xy 54.61 134.62))
+  (wire (pts (xy 54.61 104.14) (xy 54.61 132.08))
     (stroke (width 0) (type default))
   )
@@
     (stroke (width 0) (type default))
   )
+  (wire (pts (xy 54.61 132.08) (xy 71.12 132.08))
+    (stroke (width 0) (type default))
+  )
   (wire (pts (xy 194.31 121.92) (xy 203.2 121.92))
     (stroke (width 0) (type default))
@@
     (stroke (width 0) (type default))
   )
-  (wire (pts (xy 57.15 132.08) (xy 71.12 132.08))
-    (stroke (width 0) (type default))
-  )
   (wire (pts (xy 125.73 104.14) (xy 54.61 104.14))
     (stroke (width 0) (type default))
@@
     (stroke (width 0) (type default))
   )
+  (wire (pts (xy 194.31 40.64) (xy 194.31 43.18))
+    (stroke (width 0) (type default))
+  )
+  (wire (pts (xy 42.926 46.99) (xy 55.118 46.99))
+    (stroke (width 0) (type default))
+  )
+  (wire (pts (xy 161.29 144.78) (xy 171.45 144.78))
+    (stroke (width 0) (type default))
+  )
+  (wire (pts (xy 135.636 40.64) (xy 135.636 43.18))
+    (stroke (width 0) (type default))
+  )
+  (wire (pts (xy 126.746 40.64) (xy 135.636 40.64))
+    (stroke (width 0) (type default))
+  )
+  (wire (pts (xy 120.65 172.72) (xy 124.46 172.72))
+    (stroke (width 0) (type default))
+  )
+  (wire (pts (xy 123.19 121.92) (xy 123.19 106.68))
+    (stroke (width 0) (type default))
+  )
+  (wire (pts (xy 42.926 39.37) (xy 55.372 39.37))
+    (stroke (width 0) (type default))
+  )
+  (wire (pts (xy 125.73 124.46) (xy 125.73 104.14))
+    (stroke (width 0) (type default))
+  )
+  (wire (pts (xy 185.42 40.64) (xy 194.31 40.64))
+    (stroke (width 0) (type default))
+  )
+  (wire (pts (xy 194.31 65.532) (xy 194.31 68.072))
+    (stroke (width 0) (type default))
+  )
+  (wire (pts (xy 92.71 182.88) (xy 95.25 182.88))
+    (stroke (width 0) (type default))
+  )
+  (wire (pts (xy 194.31 35.306) (xy 194.31 40.64))
+    (stroke (width 0) (type default))
+  )
+  (wire (pts (xy 68.58 124.46) (xy 71.12 124.46))
+    (stroke (width 0) (type default))
+  )
+  (wire (pts (xy 177.8 75.692) (xy 194.31 75.692))
+    (stroke (width 0) (type default))
+  )
+  (wire (pts (xy 135.636 75.692) (xy 135.636 73.152))
+    (stroke (width 0) (type default))
+  )
+  (wire (pts (xy 106.68 127) (xy 123.19 127))
+    (stroke (width 0) (type default))
+  )
+  (wire (pts (xy 42.672 81.534) (xy 56.642 81.534))
+    (stroke (width 0) (type default))
+  )
+  (wire (pts (xy 176.53 110.49) (xy 186.69 110.49))
+    (stroke (width 0) (type default))
+  )
+  (wire (pts (xy 42.926 44.45) (xy 55.372 44.45))
+    (stroke (width 0) (type default))
+  )
+  (wire (pts (xy 106.68 147.32) (xy 109.22 147.32))
+    (stroke (width 0) (type default))
+  )
+  (wire (pts (xy 176.53 144.78) (xy 186.69 144.78))
+    (stroke (width 0) (type default))
+  )
+  (wire (pts (xy 38.1 185.42) (xy 41.91 185.42))
+    (stroke (width 0) (type default))
+  )
+  (wire (pts (xy 135.636 50.8) (xy 144.78 50.8))
+    (stroke (width 0) (type default))
+  )
+  (wire (pts (xy 57.15 134.62) (xy 71.12 134.62))
+    (stroke (width 0) (type default))
+  )
+  (wire (pts (xy 161.29 121.92) (xy 171.45 121.92))
+    (stroke (width 0) (type default))
+  )
+  (wire (pts (xy 120.65 167.64) (xy 120.65 172.72))
+    (stroke (width 0) (type default))
+  )
   (wire (pts (xy 68.58 127) (xy 71.12 127))
     (stroke (width 0) (type default))
   )
-  (wire (pts (xy 194.31 40.64) (xy 194.31 43.18))
-    (stroke (width 0) (type default))
-  )
-  (wire (pts (xy 42.926 46.99) (xy 55.118 46.99))
-    (stroke (width 0) (type default))
-  )
-  (wire (pts (xy 161.29 144.78) (xy 171.45 144.78))
-    (stroke (width 0) (type default))
-  )
-  (wire (pts (xy 135.636 40.64) (xy 135.636 43.18))
-    (stroke (width 0) (type default))
-  )
-  (wire (pts (xy 126.746 40.64) (xy 135.636 40.64))
-    (stroke (width 0) (type default))
-  )
-  (wire (pts (xy 120.65 172.72) (xy 124.46 172.72))
-    (stroke (width 0) (type default))
-  )
-  (wire (pts (xy 123.19 121.92) (xy 123.19 106.68))
-    (stroke (width 0) (type default))
-  )
-  (wire (pts (xy 42.926 39.37) (xy 55.372 39.37))
-    (stroke (width 0) (type default))
-  )
-  (wire (pts (xy 125.73 124.46) (xy 125.73 104.14))
-    (stroke (width 0) (type default))
-  )
-  (wire (pts (xy 185.42 40.64) (xy 194.31 40.64))
-    (stroke (width 0) (type default))
-  )
-  (wire (pts (xy 194.31 65.532) (xy 194.31 68.072))
-    (stroke (width 0) (type default))
-  )
-  (wire (pts (xy 92.71 182.88) (xy 95.25 182.88))
-    (stroke (width 0) (type default))
-  )
-  (wire (pts (xy 194.31 35.306) (xy 194.31 40.64))
-    (stroke (width 0) (type default))
-  )
-  (wire (pts (xy 54.61 134.62) (xy 71.12 134.62))
-    (stroke (width 0) (type default))
-  )
-  (wire (pts (xy 177.8 75.692) (xy 194.31 75.692))
-    (stroke (width 0) (type default))
-  )
-  (wire (pts (xy 68.58 124.46) (xy 71.12 124.46))
-    (stroke (width 0) (type default))
-  )
-  (wire (pts (xy 135.636 75.692) (xy 135.636 73.152))
-    (stroke (width 0) (type default))
-  )
-  (wire (pts (xy 106.68 127) (xy 123.19 127))
-    (stroke (width 0) (type default))
-  )
-  (wire (pts (xy 68.58 121.92) (xy 71.12 121.92))
-    (stroke (width 0) (type default))
-  )
-  (wire (pts (xy 42.672 81.534) (xy 56.642 81.534))
-    (stroke (width 0) (type default))
-  )
-  (wire (pts (xy 176.53 110.49) (xy 186.69 110.49))
-    (stroke (width 0) (type default))
-  )
-  (wire (pts (xy 42.926 44.45) (xy 55.372 44.45))
-    (stroke (width 0) (type default))
-  )
-  (wire (pts (xy 106.68 147.32) (xy 109.22 147.32))
-    (stroke (width 0) (type default))
-  )
-  (wire (pts (xy 176.53 144.78) (xy 186.69 144.78))
+  (wire (pts (xy 41.91 170.18) (xy 43.18 170.18))
+    (stroke (width 0) (type default))
+  )
+  (wire (pts (xy 41.91 167.64) (xy 43.18 167.64))
+    (stroke (width 0) (type default))
+  )
+  (wire (pts (xy 129.54 172.72) (xy 133.35 172.72))
+    (stroke (width 0) (type default))
+  )
+  (wire (pts (xy 123.19 106.68) (xy 57.15 106.68))
+    (stroke (width 0) (type default))
+  )
+  (wire (pts (xy 119.126 75.692) (xy 135.636 75.692))
+    (stroke (width 0) (type default))
+  )
+  (wire (pts (xy 135.636 50.8) (xy 135.636 48.26))
     (stroke (width 0) (type default))
   )
   (wire (pts (xy 68.58 129.54) (xy 71.12 129.54))
-    (stroke (width 0) (type default))
-  )
-  (wire (pts (xy 38.1 185.42) (xy 41.91 185.42))
-    (stroke (width 0) (type default))
-  )
-  (wire (pts (xy 135.636 50.8) (xy 144.78 50.8))
-    (stroke (width 0) (type default))
-  )
-  (wire (pts (xy 161.29 121.92) (xy 171.45 121.92))
-    (stroke (width 0) (type default))
-  )
-  (wire (pts (xy 120.65 167.64) (xy 120.65 172.72))
-    (stroke (width 0) (type default))
-  )
-  (wire (pts (xy 41.91 170.18) (xy 43.18 170.18))
-    (stroke (width 0) (type default))
-  )
-  (wire (pts (xy 41.91 167.64) (xy 43.18 167.64))
-    (stroke (width 0) (type default))
-  )
-  (wire (pts (xy 129.54 172.72) (xy 133.35 172.72))
-    (stroke (width 0) (type default))
-  )
-  (wire (pts (xy 123.19 106.68) (xy 57.15 106.68))
-    (stroke (width 0) (type default))
-  )
-  (wire (pts (xy 119.126 75.692) (xy 135.636 75.692))
-    (stroke (width 0) (type default))
-  )
-  (wire (pts (xy 57.15 106.68) (xy 57.15 132.08))
-    (stroke (width 0) (type default))
-  )
-  (wire (pts (xy 135.636 50.8) (xy 135.636 48.26))
     (stroke (width 0) (type default))
   )
@@
     (effects (font (size 1.27 1.27)) (justify right))
   )
-  (hierarchical_label "CON_2" (shape input) (at 68.58 124.46 180) (fields_autoplaced)
+  (hierarchical_label "CON_2" (shape input) (at 68.58 127 180) (fields_autoplaced)
     (effects (font (size 1.27 1.27)) (justify right))
   )
-  (hierarchical_label "CON_1" (shape input) (at 68.58 121.92 180) (fields_autoplaced)
+  (hierarchical_label "CON_1" (shape input) (at 68.58 129.54 180) (fields_autoplaced)
     (effects (font (size 1.27 1.27)) (justify right))
   )
-  (hierarchical_label "CON_4" (shape input) (at 68.58 129.54 180) (fields_autoplaced)
+  (hierarchical_label "CON_4" (shape input) (at 68.58 121.92 180) (fields_autoplaced)
     (effects (font (size 1.27 1.27)) (justify right))
   )
@@
     (effects (font (size 1.27 1.27)) (justify right))
   )
-  (hierarchical_label "CON_3" (shape input) (at 68.58 127 180) (fields_autoplaced)
+  (hierarchical_label "CON_3" (shape input) (at 68.58 124.46 180) (fields_autoplaced)
     (effects (font (size 1.27 1.27)) (justify right))
   )
@@
       (project "bms"
         (path "/e0ec80f6-0ac5-448e-a052-7eb38c8b1976"
-          (reference "R13") (unit 1)
-        )
-      )
+          (reference "R11") (unit 1)
+        )
+      )
