File: boards/Arduino Shield/Arduino Shield.kicad_sch (KiCad schematic)
At the start: 1 part

Commit message: Remove resistor
Parts:
- removed R1: R, symbol Device:R
Changed lines of the file:
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@@
 (kicad_sch (version 20230121) (generator eeschema)
   (paper "A4")
-  (symbol (lib_id "Device:R") (at 50.8 46.99 0) (unit 1)
-    (in_bom yes) (on_board yes) (dnp no) (fields_autoplaced)
-    (property "Reference" "R1" (at 53.34 45.72 0)
-      (effects (font (size 1.27 1.27)) (justify left))
-    )
-    (property "Value" "R" (at 53.34 48.26 0)
-      (effects (font (size 1.27 1.27)) (justify left))
-    )
-    (property "Footprint" "" (at 49.022 46.99 90)
-      (effects (font (size 1.27 1.27)) hide)
-    )
-    (property "Datasheet" "~" (at 50.8 46.99 0)
-      (effects (font (size 1.27 1.27)) hide)
-    )
-    (pin "1")
-    (pin "2")
-    (instances
-      (project "Arduino Shield"
-        (path "/d7e93cbd-19df-457a-85c5-e42e2ae79e40"
-          (reference "R1") (unit 1)
-        )
-      )
-    )
-  )
   (sheet_instances
     (path "/" (page "1"))
