File: boards/PCBPCBNEW/PCBPCBNEW.kicad_pcb (KiCad board)
At the start: 4 copper layers, 79 parts, among them J1 Screw_Terminal_01x02, J4 Screw_Terminal_01x06, U1 SIC431AED-T1-GE3, U2 SIC431AED-T1-GE3, U3 SIC431AED-T1-GE3

Commit message: GL
Parts:
- L1, L2, L3: value 1uH -> 1.2uH
- R16, R17, R18: value 0 -> 3.3
- R22, R23: value 78.7k -> 73.2
- R24: value 78.7k -> 73.2k
Connections:
- U1 pad 10: /GL -> unconnected-(U1-GL-Pad10)
- U1 pad 11: /GL -> unconnected-(U1-GL-Pad10)_2
- U1 pad 28: /GL -> unconnected-(U1-GL-Pad10)_1
- U2 pad 10: /GL -> unconnected-(U2-GL-Pad10)_2
- U2 pad 11: /GL -> unconnected-(U2-GL-Pad10)
- U2 pad 28: /GL -> unconnected-(U2-GL-Pad10)_1
- U3 pad 10: /GL -> unconnected-(U3-GL-Pad10)_1
- U3 pad 11: /GL -> unconnected-(U3-GL-Pad10)_2
- U3 pad 28: /GL -> unconnected-(U3-GL-Pad10)
Routing:
- net /GL: track 9.65 -> 0.00 mm
