File: boards/PCBPCBNEW2/PCBPCBNEW.kicad_pcb (KiCad board)
At the start: 4 copper layers, 0 parts

Commit message: Remade schematic and imported library
Parts:
- added C1: 150uF, Capacitor_THT:CP_Radial_D12.5mm_P5.00mm, F.Cu at (183.6, 89.4)
- added C10: 47uF, Capacitor_SMD:C_0805_2012Metric, F.Cu at (199.8, 116.2)
- added C11: 47uF, Capacitor_SMD:C_0805_2012Metric, F.Cu at (199.8, 119.2)
- added C12: 47uF, Capacitor_SMD:C_0805_2012Metric, F.Cu at (199.8, 122.2)
- added C13: 150uF, Capacitor_THT:CP_Radial_D12.5mm_P5.00mm, F.Cu at (183.6, 103.5)
- added C14: 100nF, Capacitor_SMD:C_0805_2012Metric, F.Cu at (199.8, 125.2)
- added C15: 1uF, Capacitor_SMD:C_0805_2012Metric, F.Cu at (199.8, 128.2)
- added C16: 100nF, Capacitor_SMD:C_0805_2012Metric, F.Cu at (199.8, 131.2)
- added C17: 4.7uF, Capacitor_SMD:C_0805_2012Metric, F.Cu at (204.3, 113.1)
- added C18: 100nF, Capacitor_SMD:C_0805_2012Metric, F.Cu at (204.3, 116.2)
- added C19: 47uF, Capacitor_SMD:C_0805_2012Metric, F.Cu at (204.3, 119.2)
- added C2: 100nF, Capacitor_SMD:C_0805_2012Metric, F.Cu at (195.4, 113.1)
- added C20: 47uF, Capacitor_SMD:C_0805_2012Metric, F.Cu at (204.3, 122.2)
- added C21: 47uF, Capacitor_SMD:C_0805_2012Metric, F.Cu at (204.3, 125.2)
- added C22: 47uF, Capacitor_SMD:C_0805_2012Metric, F.Cu at (204.3, 128.2)
- added C23: 47uF, Capacitor_SMD:C_0805_2012Metric, F.Cu at (204.3, 131.2)
- added C24: 47uF, Capacitor_SMD:C_0805_2012Metric, F.Cu at (208.7, 113.1)
- added C25: 100nF, Capacitor_SMD:C_0805_2012Metric, F.Cu at (208.7, 116.2)
- added C3: 1uF, Capacitor_SMD:C_0805_2012Metric, F.Cu at (195.4, 116.2)
- added C32: 47uF, Capacitor_SMD:C_0805_2012Metric, F.Cu at (208.7, 119.2)
- added C39: 47uF, Capacitor_SMD:C_0805_2012Metric, F.Cu at (208.7, 122.2)
- added C4: 100nF, Capacitor_SMD:C_0805_2012Metric, F.Cu at (195.4, 119.2)
- added C40: 47uF, Capacitor_SMD:C_0805_2012Metric, F.Cu at (208.7, 125.2)
- added C41: 47uF, Capacitor_SMD:C_0805_2012Metric, F.Cu at (208.7, 128.2)
- added C42: 47uF, Capacitor_SMD:C_0805_2012Metric, F.Cu at (208.7, 131.2)
- added C43: 47uF, Capacitor_SMD:C_0805_2012Metric, F.Cu at (213.2, 113.1)
- added C44: 100nF, Capacitor_SMD:C_0805_2012Metric, F.Cu at (213.2, 116.2)
- added C45: 1uF, Capacitor_SMD:C_0805_2012Metric, F.Cu at (213.2, 119.2)
- added C46: 4.7uF, Capacitor_SMD:C_0805_2012Metric, F.Cu at (213.2, 122.2)
- added C47: 150uF, Capacitor_THT:CP_Radial_D12.5mm_P5.00mm, F.Cu at (183.6, 117.5)
- added C48: 100nF, Capacitor_SMD:C_0805_2012Metric, F.Cu at (213.2, 125.2)
- added C5: 4.7uF, Capacitor_SMD:C_0805_2012Metric, F.Cu at (195.4, 122.2)
- added C6: 100nF, Capacitor_SMD:C_0805_2012Metric, F.Cu at (195.4, 125.2)
- added C7: 47uF, Capacitor_SMD:C_0805_2012Metric, F.Cu at (195.4, 128.2)
- added C8: 47uF, Capacitor_SMD:C_0805_2012Metric, F.Cu at (195.4, 131.2)
- added C9: 47uF, Capacitor_SMD:C_0805_2012Metric, F.Cu at (199.8, 113.1)
- added F1: 0685P9200-01, 0685P9200_01:FUSC3215X83N, F.Cu at (225.1, 93.3)
- added F2: 0685P9200-01, 0685P9200_01:FUSC3215X83N, F.Cu at (225.1, 96.8)
- added F3: 0685P9200-01, 0685P9200_01:FUSC3215X83N, F.Cu at (225.1, 100.3)
- added J1: Screw_Terminal_01x02, REAAAL:TE_1986660-2a, F.Cu at (199.6, 94.0)
- added J4: Screw_Terminal_01x06, REAAAL:TEST2, F.Cu at (209.0, 86.7)
- added L1: 1.2uH, Inductor_SMD:L_Vishay_IHLP-5050, F.Cu at (170.6, 89.5)
- added L2: 1.2uH, Inductor_SMD:L_Vishay_IHLP-5050, F.Cu at (170.6, 103.8)
- added L4: 1.2uH, Inductor_SMD:L_Vishay_IHLP-5050, F.Cu at (170.6, 118.0)
- added R1: 562k, Resistor_SMD:R_0805_2012Metric, F.Cu at (217.6, 113.1)
- added R10: 309k, Resistor_SMD:R_0805_2012Metric, F.Cu at (222.0, 119.0)
- added R11: 200k, Resistor_SMD:R_0805_2012Metric, F.Cu at (222.0, 122.0)
- added R12: 100k, Resistor_SMD:R_0805_2012Metric, F.Cu at (222.0, 124.9)
- added R13: 3.3, Resistor_SMD:R_0805_2012Metric, F.Cu at (222.0, 127.9)
- added R14: 100k, Resistor_SMD:R_0805_2012Metric, F.Cu at (222.0, 130.8)
- added R15: 10k, Resistor_SMD:R_0805_2012Metric, F.Cu at (226.4, 113.1)
- added R16: 73.2, Resistor_SMD:R_0805_2012Metric, F.Cu at (226.4, 116.1)
- added R2: 309k, Resistor_SMD:R_0805_2012Metric, F.Cu at (217.6, 116.1)
- added R25: 3.3, Resistor_SMD:R_0805_2012Metric, F.Cu at (226.4, 119.0)
- added R26: 10k, Resistor_SMD:R_0805_2012Metric, F.Cu at (226.4, 122.0)
- added R27: 73.2, Resistor_SMD:R_0805_2012Metric, F.Cu at (226.4, 124.9)
- added R28: 100k, Resistor_SMD:R_0805_2012Metric, F.Cu at (226.4, 127.9)
- added R29: 100k, Resistor_SMD:R_0805_2012Metric, F.Cu at (226.4, 130.8)
- added R3: 200k, Resistor_SMD:R_0805_2012Metric, F.Cu at (217.6, 119.0)
- added R30: 200k, Resistor_SMD:R_0805_2012Metric, F.Cu at (230.8, 113.1)
- added R31: 562k, Resistor_SMD:R_0805_2012Metric, F.Cu at (230.8, 116.1)
- added R32: 309k, Resistor_SMD:R_0805_2012Metric, F.Cu at (230.8, 119.0)
- added R4: 100k, Resistor_SMD:R_0805_2012Metric, F.Cu at (217.6, 122.0)
- added R5: 3.3, Resistor_SMD:R_0805_2012Metric, F.Cu at (217.6, 124.9)
- added R6: 100k, Resistor_SMD:R_0805_2012Metric, F.Cu at (217.6, 127.9)
- added R7: 10k, Resistor_SMD:R_0805_2012Metric, F.Cu at (217.6, 130.8)
- added R8: 73.2, Resistor_SMD:R_0805_2012Metric, F.Cu at (222.0, 113.1)
- added R9: 562k, Resistor_SMD:R_0805_2012Metric, F.Cu at (222.0, 116.1)
- added U1: SIC431AED-T1-GE3, SIC431AED_T1_GE3:REGULATOR_SIC431AED-T1-GE3, F.Cu at (219.1, 94.7)
- added U2: SIC431AED-T1-GE3, SIC431AED_T1_GE3:REGULATOR_SIC431AED-T1-GE3, F.Cu at (219.1, 100.8)
- added U4: SIC431AED-T1-GE3, SIC431AED_T1_GE3:REGULATOR_SIC431AED-T1-GE3, F.Cu at (219.1, 107.0)
