File: boards/12V10A Stepdown/converter/converter.kicad_pcb (KiCad board)
At the start: 2 copper layers, 27 parts, among them J1 TB005-762-02BE, J2 TB005-762-02BE, M1 CSD17578Q3A, M2 CSD17571Q2, U1 LM25145RGYR

Commit message: pcbfirst
Parts:
- moved J1 68.1 mm to (59.4, 87.6), turned to 180 degrees
- moved J2 66.1 mm to (76.6, 87.7), turned to 180 degrees
- moved Rcomp1 49.8 mm to (55.7, 69.9)
- moved Cout1 30.4 mm to (74.1, 74.5)
- moved Cin1 26.9 mm to (55.6, 73.6)
- moved 2.2uH1 25.1 mm to (73.5, 66.7), turned to -90 degrees
- moved Rcomp2 24.3 mm to (69.3, 74.2), turned to -90 degrees
- moved Cilim1 22.7 mm to (62.5, 73.6)
- moved Rfbb1 21.3 mm to (66.1, 74.1), turned to 90 degrees
- moved Rvcc1 19.5 mm to (61.9, 75.8)
- moved Ccomp1 19.4 mm to (55.7, 68.5), turned to 180 degrees
- moved Rfbt1 17.9 mm to (67.7, 73.9), turned to -90 degrees
- moved U1 17.1 mm to (62.3, 69.9)
- moved Ccomp2 17.0 mm to (57.7, 69.4), turned to -90 degrees
- moved Rilim1 16.1 mm to (64.6, 75.6), turned to 90 degrees
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Routing:
- net GND: track 0.00 -> 92.9 mm
- net Net-(U1-VCC): track 0.00 -> 33.2 mm, vias 0 -> 3
- net Net-(M1-D5): track 0.00 -> 31.8 mm, vias 0 -> 2
- net Net-(2.2uH1-Pad2): track 0.00 -> 30.8 mm, vias 0 -> 2
- net Net-(U1-FB): track 0.00 -> 24.8 mm, vias 0 -> 2
- net Net-(U1-VIN): track 0.00 -> 17.5 mm
- net Net-(U1-PGOOD): track 0.00 -> 12.1 mm, vias 0 -> 2
- net Net-(M1-S1): track 0.00 -> 11.1 mm
- net Net-(U1-EN/UVLO): track 0.00 -> 10.9 mm
- net Net-(U1-RT): track 0.00 -> 8.54 mm
- net Net-(U1-ILIM): track 0.00 -> 7.08 mm
- net Net-(U1-SS/TRK): track 0.00 -> 6.43 mm, vias 0 -> 2
- net Net-(U1-SYNCIN): track 0.00 -> 5.96 mm
- net Net-(U1-COMP): track 0.00 -> 4.97 mm
- net Net-(M1-G): track 0.00 -> 4.67 mm
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